File: crates/backend-kicad/tests/golden/board/connectors/golden.kicad_pcb (KiCad board)
At the start: 2 copper layers, 100 x 80 mm, 4 parts, among them J1 J, J2 J, J3 J, J4 J

Commit message: Fix bugs with footprints and DRC rules
Other:
- net class Default: trace_width 0.25 -> 0.2
Changed lines of the file:
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@@
   (net_class "Default" ""
     (clearance 0.2)
-    (trace_width 0.25)
+    (trace_width 0.2)
     (via_dia 0.8)
     (via_drill 0.4)
