File: crates/backend-kicad/tests/golden/board/passives/golden.kicad_pcb (KiCad board)
At the start: 2 copper layers, 100 x 80 mm, 5 parts, among them Y1 Y

Commit message: Apply stabilise-copperleaf-pipeline
Parts:
- C1: footprint Capacitor_SMD.3dshapes/C_0603_1608Metric -> Capacitor_SMD:C_0603_1608Metric
- R1: footprint Resistor_SMD.3dshapes/R_0603_1608Metric -> Resistor_SMD:R_0603_1608Metric
Changed lines of the file:
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@@
     (layer "Edge.Cuts")
 )
-  (footprint "Capacitor_SMD.3dshapes/C_0603_1608Metric"
+  (footprint "Capacitor_SMD:C_0603_1608Metric"
     (layer "F.Cu")
     (locked no)
@@
       (rotate
         (xyz 0 0 0))))
-  (footprint "Resistor_SMD.3dshapes/R_0603_1608Metric"
+  (footprint "Resistor_SMD:R_0603_1608Metric"
     (layer "F.Cu")
     (locked no)
