File: crates/backend-kicad/tests/golden/board/passives/golden.kicad_sch (KiCad schematic)
At the start: 5 parts, among them Y1 Y

Commit message: Improve recognition of bypass caps
Parts:
- C1: value C -> 100nF; symbol copperleaf:C1 -> copperleaf:Capacitor
Changed lines of the file:
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@@
     (date ""))
   (symbol
-    (lib_id "copperleaf:C1")
+    (lib_id "copperleaf:Capacitor")
     (at 35.56 33.02 0)
     (unit 1)
@@
         (font
           (size 1.27 1.27))))
-    (property "Value" "C"
+    (property "Value" "100nF"
       (at 35.56 36.83 0)
       (effects

Commit message: Apply stabilise-copperleaf-pipeline
Parts:
- C1: footprint Capacitor_SMD.3dshapes/C_0603_1608Metric -> Capacitor_SMD:C_0603_1608Metric
- R1: footprint Resistor_SMD.3dshapes/R_0603_1608Metric -> Resistor_SMD:R_0603_1608Metric
Changed lines of the file:
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@@
         (font
           (size 1.27 1.27))))
-    (property "Footprint" "Capacitor_SMD.3dshapes/C_0603_1608Metric"
+    (property "Footprint" "Capacitor_SMD:C_0603_1608Metric"
       (at 35.56 33.02 0)
       (hide yes)
@@
         (font
           (size 1.27 1.27))))
-    (property "Footprint" "Resistor_SMD.3dshapes/R_0603_1608Metric"
+    (property "Footprint" "Resistor_SMD:R_0603_1608Metric"
       (at 68.58 33.02 0)
       (hide yes)
