File: crates/backend-kicad/tests/golden/board/raspberrypi/golden.kicad_pcb (KiCad board)
At the start: 2 copper layers, 100 x 80 mm, 3 parts, among them U1 U

Commit message: Apply stabilise-copperleaf-pipeline
Parts:
- C1, C2: footprint Capacitor_SMD.3dshapes/C_0603_1608Metric -> Capacitor_SMD:C_0603_1608Metric
Changed lines of the file:
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@@
       (rotate
         (xyz 0 0 0))))
-  (footprint "Capacitor_SMD.3dshapes/C_0603_1608Metric"
+  (footprint "Capacitor_SMD:C_0603_1608Metric"
     (layer "F.Cu")
     (locked no)
@@
       (rotate
         (xyz 0 0 0))))
-  (footprint "Capacitor_SMD.3dshapes/C_0603_1608Metric"
+  (footprint "Capacitor_SMD:C_0603_1608Metric"
     (layer "F.Cu")
     (locked no)
